File: pcb/PCBEasyEDA.kicad_sch (KiCad schematic)
At the start: 56 parts

Commit message: maybe
Parts:
- +, -, PIEZO+, PIEZO+1, PIEZO+2, PIEZO+3, PIEZO+4, PIEZO+5, PIEZO+6, PIEZO+7, PIEZO-, PIEZO-1, PIEZO-2, PIEZO-3, PIEZO-4, PIEZO-5, PIEZO-6, PIEZO-7: footprint (none) -> THROUGHHOLEPIN
- 100K1, 100K2, 100K3, 100K4, 100K5, 100K6, 100K7, 100K8, 100NF, 100NF2, 1K1, 1K2, 1K3, 1K4, 1K5, 1K6, 1K7, 1K8: footprint (none) -> 0207/10
- 10UF: footprint (none) -> 10UF 100V
- 74HC595: footprint (none) -> 74HC595
- ARDUINO_NANO: footprint (none) -> COMM-TH_ARDUINO_NANO
- DIODE1, DIODE2, DIODE3, DIODE4, DIODE5, DIODE6, DIODE7, DIODE8: footprint (none) -> 1N4007_(DO-41)
- FUSE1: footprint (none) -> POLYFUSE FOOTPRINT
- MOSFET1, MOSFET2, MOSFET3, MOSFET4, MOSFET5, MOSFET6, MOSFET7, MOSFET8: footprint (none) -> TO-220AB-3_L10.4-W4.6-P2.54-L
Other:
- moved on the sheet: +, -, 100K1, 100K2, 100K3, 100K4, 100K5, 100K6, 100K7, 100K8, 100NF, 100NF2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

Commit message: aaaaaaaaa
Other:
- note removed: "#10: Info: symbol for PIEZO-1 (rotation:0) exits as PIEZO+_AE02EF48"
- note removed: "#11: Info: symbol for PIEZO+1 (rotation:0) exits as PIEZO+_AE02EF48"
- note removed: "#12: Info: symbol for MOSFET2 (rotation:0) exits as MOSFET_41B7232A"
- note removed: "#13: Info: symbol for 1K1 (rotation:0) is new as K_63839ECC"
- note removed: "#14: Info: symbol for 1K2 (rotation:0) exits as K_63839ECC"
- note removed: "#15: Info: symbol for DIODE1 (rotation:90) is new as DIODE_AC9B690"
- note removed: "#16: Info: symbol for DIODE2 (rotation:90) exits as DIODE_AC9B690"
- note removed: "#17: Info: symbol for 1K3 (rotation:0) exits as K_63839ECC"
- note removed: "#18: Info: symbol for MOSFET3 (rotation:0) exits as MOSFET_41B7232A"
- note removed: "#19: Info: symbol for PIEZO+2 (rotation:0) exits as PIEZO+_AE02EF48"
- note removed: "#1: Info: below are the conversion remarks. The conversion may contain errors. Please read the remarks carefully and run the ERC check to solve issues. To find a component mentioned in the remarks go to: Kicad menu Edit > Find and enter the EDA_id (gge....); search for hidden fields. Only the id of the symbol can be found; the id of the shape is in the input json."
- note removed: "#20: Info: symbol for DIODE3 (rotation:90) exits as DIODE_AC9B690"
- note removed: "#21: Info: symbol for PIEZO-2 (rotation:0) exits as PIEZO+_AE02EF48"
- note removed: "#22: Info: symbol for PIEZO+3 (rotation:0) exits as PIEZO+_AE02EF48"
- note removed: "#23: Info: symbol for DIODE4 (rotation:90) exits as DIODE_AC9B690"
- note removed: "#24: Info: symbol for PIEZO-3 (rotation:0) exits as PIEZO+_AE02EF48"
- note removed: "#25: Info: symbol for 1K4 (rotation:0) exits as K_63839ECC"
- note removed: "#26: Info: symbol for MOSFET4 (rotation:0) exits as MOSFET_41B7232A"
- note removed: "#27: Info: symbol for 1K5 (rotation:0) exits as K_63839ECC"
- note removed: "#28: Info: symbol for MOSFET5 (rotation:0) exits as MOSFET_41B7232A"
- note removed: "#29: Info: symbol for PIEZO+4 (rotation:0) exits as PIEZO+_AE02EF48"
- note removed: "#2: Warning: unsupported shape ellipse found in schematics; shape ignored"
- note removed: "#30: Info: symbol for PIEZO-4 (rotation:0) exits as PIEZO+_AE02EF48"
- note removed: "#31: Info: symbol for DIODE5 (rotation:90) exits as DIODE_AC9B690"
- note removed: "#32: Info: symbol for DIODE6 (rotation:90) exits as DIODE_AC9B690"
- note removed: "#33: Info: symbol for PIEZO+5 (rotation:0) exits as PIEZO+_AE02EF48"
- note removed: "#34: Info: symbol for PIEZO-5 (rotation:0) exits as PIEZO+_AE02EF48"
- note removed: "#35: Info: symbol for 1K6 (rotation:0) exits as K_63839ECC"
- note removed: "#36: Info: symbol for MOSFET6 (rotation:0) exits as MOSFET_41B7232A"
- note removed: "#37: Info: symbol for 1K7 (rotation:0) exits as K_63839ECC"
- note removed: "#38: Info: symbol for MOSFET7 (rotation:0) exits as MOSFET_41B7232A"
- note removed: "#39: Info: symbol for PIEZO+6 (rotation:0) exits as PIEZO+_AE02EF48"
- note removed: "#3: Info: symbol for ARDUINO_NANO (rotation:0) is new as ARDUINO_NANO_338AB957"
- note removed: "#40: Info: symbol for DIODE7 (rotation:90) exits as DIODE_AC9B690"
- note removed: "#41: Info: symbol for PIEZO-6 (rotation:0) exits as PIEZO+_AE02EF48"
- note removed: "#42: Info: symbol for DIODE8 (rotation:90) exits as DIODE_AC9B690"
- note removed: "#43: Info: symbol for PIEZO+7 (rotation:0) exits as PIEZO+_AE02EF48"
- note removed: "#44: Info: symbol for PIEZO-7 (rotation:0) exits as PIEZO+_AE02EF48"
- note removed: "#45: Info: symbol for 1K8 (rotation:0) exits as K_63839ECC"
- note removed: "#46: Info: symbol for MOSFET8 (rotation:0) exits as MOSFET_41B7232A"
- note removed: "#47: Info: symbol for 100NF (rotation:270) is new as NF_779C8389"
- note removed: "#48: Info: symbol for 100NF2 (rotation:0) exits as K_63839ECC"
- note removed: "#49: Info: symbol for 10UF (rotation:270) is new as UF_FBF4E86A"
- note removed: "#4: Info: symbol for 74HC595 (rotation:0) is new as HC_F2BFCCF1"
- note removed: "#50: Info: symbol for 100K1 (rotation:90) is new as K_EA51191F"
- note removed: "#51: Info: symbol for 100K2 (rotation:0) exits as K_63839ECC"
- note removed: "#52: Info: symbol for 100K3 (rotation:90) exits as K_EA51191F"
- note removed: "#53: Info: symbol for 100K4 (rotation:90) exits as K_EA51191F"
- note removed: "#54: Info: symbol for 100K5 (rotation:90) exits as K_EA51191F"
- note removed: "#55: Info: symbol for 100K6 (rotation:90) exits as K_EA51191F"
- note removed: "#56: Info: symbol for 100K7 (rotation:90) exits as K_EA51191F"
- note removed: "#57: Info: symbol for 100K8 (rotation:90) exits as K_EA51191F"
- note removed: "#58: Info: symbol for FUSE1 (rotation:0) is new as FUSE_AE3E1684"
- note removed: "#5: Info: symbol for - (rotation:180) is new as -_4FD4D7A7"
- note removed: "#6: Info: symbol for + (rotation:180) exits as -_4FD4D7A7"
- note removed: "#7: Info: symbol for MOSFET1 (rotation:0) is new as MOSFET_41B7232A"
- note removed: "#8: Info: symbol for PIEZO+ (rotation:0) is new as PIEZO+_AE02EF48"
- note removed: "#9: Info: symbol for PIEZO- (rotation:0) exits as PIEZO+_AE02EF48"
